File: drone_v3/Power_supply.sch (KiCad schematic (older format))
At the start: 16 parts, among them U9 MCP1700-3302E_SOT23

Commit message: add alot
Parts:
- D1: footprint Diode_SMD:D_0805_2012Metric_Pad1.15x1.40mm_HandSolder -> Diode_SMD:D_1206_3216Metric
Connections:
- net PWR_IN: now reaches C15.1, C16.1, C17.1, D1.2 (A), U9.3 (VI)
Changed lines of the file:
@@
 F 0 "D1" V 3554 4228 50  0000 L CNN
 F 1 "DIODE" V 3645 4228 50  0000 L CNN
-F 2 "Diode_SMD:D_0805_2012Metric_Pad1.15x1.40mm_HandSolder" H 3600 4100 50  0001 C CNN
+F 2 "Diode_SMD:D_1206_3216Metric" H 3600 4100 50  0001 C CNN
 F 3 "~" H 3600 4100 50  0001 C CNN
 	1    3600 4100
@@
 	1    0    0    -1
 $EndComp
+Text GLabel 3300 4300 0    50   Input ~ 0
+PWR_IN
+Wire Wire Line
+	3300 4300 3600 4300
 $EndSCHEMATC
