File: drone_v3/IMU.sch (KiCad schematic (older format))
At the start: 15 parts, among them J2 Conn_01x10_Female, U3 MPU-9250, U7 MS5611-01BA, U8 ICM-20602

Commit message: add alot
Parts:
- removed C27: C, Capacitor_SMD:C_0603_1608Metric, symbol Device:C
- added C29, C30: 1uF, Capacitor_SMD:C_0603_1608Metric_Pad1.05x0.95mm_HandSolder, symbol Device:C
- added U4: MCP1700-3302E_SOT23, Package_TO_SOT_SMD:SOT-23, symbol Regulator_Linear:MCP1700-3302E_SOT23
Connections:
- net GND: now also C29.2, C30.2, U4.1 (GND)
- net VCC renamed +3.3VA
- net +3.3VA: now also C30.1, U4.2 (VO)
- new net +5V: C29.1, U4.3 (VI)
Changed lines of the file:
@@
-$EndComp
-$Comp
-L power:VCC #PWR0109
-U 1 1 5F2BEBE6
-P 8250 3550
-F 0 "#PWR0109" H 8250 3400 50  0001 C CNN
-F 1 "VCC" H 8265 3723 50  0000 C CNN
-F 2 "" H 8250 3550 50  0001 C CNN
-F 3 "" H 8250 3550 50  0001 C CNN
-	1    8250 3550
-	1    0    0    -1
 $EndComp
 $Comp
@@
 Wire Wire Line
 	4750 3100 4750 3500
-$Comp
-L power:VCC #PWR0111
-U 1 1 5F2D0B30
-P 5850 3100
-F 0 "#PWR0111" H 5850 2950 50  0001 C CNN
-F 1 "VCC" H 5865 3273 50  0000 C CNN
-F 2 "" H 5850 3100 50  0001 C CNN
-F 3 "" H 5850 3100 50  0001 C CNN
-	1    5850 3100
-	1    0    0    -1
-$EndComp
 Wire Wire Line
 	5000 3350 5800 3350
@@
 Wire Wire Line
 	7750 5650 8000 5650
-$Comp
-L power:VCC #PWR0139
-U 1 1 5F2F87B9
-P 8400 5000
-F 0 "#PWR0139" H 8400 4850 50  0001 C CNN
-F 1 "VCC" H 8415 5173 50  0000 C CNN
-F 2 "" H 8400 5000 50  0001 C CNN
-F 3 "" H 8400 5000 50  0001 C CNN
-	1    8400 5000
-	1    0    0    -1
-$EndComp
 Wire Wire Line
 	8400 5000 8400 5050
@@
 	1    0    0    -1
 $EndComp
-$Comp
-L power:VCC #PWR0165
-U 1 1 5F311752
-P 2850 3000
-F 0 "#PWR0165" H 2850 2850 50  0001 C CNN
-F 1 "VCC" H 2865 3173 50  0000 C CNN
-F 2 "" H 2850 3000 50  0001 C CNN
-F 3 "" H 2850 3000 50  0001 C CNN
-	1    2850 3000
-	1    0    0    -1
-$EndComp
 Wire Wire Line
 	2750 3400 2750 3000
@@
 	1    0    0    -1
 $EndComp
-$Comp
-L Device:C C27
-U 1 1 5F345FBD
-P 7450 3450
-F 0 "C27" H 7565 3496 50  0000 L CNN
-F 1 "C" H 7565 3405 50  0000 L CNN
-F 2 "Capacitor_SMD:C_0603_1608Metric" H 7488 3300 50  0001 C CNN
-F 3 "~" H 7450 3450 50  0001 C CNN
-	1    7450 3450
-	1    0    0    -1
-$EndComp
 Wire Wire Line
 	6600 3300 7000 3300
 Connection ~ 6600 3300
-Connection ~ 7000 3300
-Wire Wire Line
-	7000 3300 7450 3300
 Wire Wire Line
 	6000 3400 6000 3300
@@
 	1    0    0    -1
 $EndComp
-$Comp
-L power:GND #PWR0170
-U 1 1 5F34C766
-P 7450 3700
-F 0 "#PWR0170" H 7450 3450 50  0001 C CNN
-F 1 "GND" H 7455 3527 50  0000 C CNN
-F 2 "" H 7450 3700 50  0001 C CNN
-F 3 "" H 7450 3700 50  0001 C CNN
-	1    7450 3700
-	1    0    0    -1
-$EndComp
-Wire Wire Line
-	7450 3600 7450 3700
 Wire Wire Line
 	7000 3600 7000 3700
+$Comp
+L Device:C C?
+U 1 1 5F35FE87
+P 2650 5850
+AR Path="/5F35FE87" Ref="C?"  Part="1"
+AR Path="/5F569749/5F35FE87" Ref="C?"  Part="1"
+AR Path="/5F3218EE/5F35FE87" Ref="C29"  Part="1"
+F 0 "C29" H 2765 5896 50  0000 L CNN
+F 1 "1uF" H 2765 5805 50  0000 L CNN
+F 2 "Capacitor_SMD:C_0603_1608Metric_Pad1.05x0.95mm_HandSolder" H 2688 5700 50  0001 C CNN
+F 3 "~" H 2650 5850 50  0001 C CNN
+	1    2650 5850
+	1    0    0    -1
+$EndComp
+$Comp
+L Device:C C?
+U 1 1 5F35FE8D
+P 3750 5850
+AR Path="/5F35FE8D" Ref="C?"  Part="1"
+AR Path="/5F569749/5F35FE8D" Ref="C?"  Part="1"
+AR Path="/5F3218EE/5F35FE8D" Ref="C30"  Part="1"
+F 0 "C30" H 3865 5896 50  0000 L CNN
+F 1 "1uF" H 3865 5805 50  0000 L CNN
+F 2 "Capacitor_SMD:C_0603_1608Metric_Pad1.05x0.95mm_HandSolder" H 3788 5700 50  0001 C CNN
+F 3 "~" H 3750 5850 50  0001 C CNN
+	1    3750 5850
+	1    0    0    -1
+$EndComp
+Wire Wire Line
+	2650 6000 3250 6000
+Wire Wire Line
+	3550 5700 3750 5700
+Wire Wire Line
+	3250 6000 3750 6000
+Connection ~ 3250 6000
+Wire Wire Line
+	3250 6000 3250 6150
+Wire Wire Line
+	2650 5700 2950 5700
+$Comp
+L Regulator_Linear:MCP1700-3302E_SOT23 U?
+U 1 1 5F35FEA1
+P 3250 5700
+AR Path="/5F569749/5F35FEA1" Ref="U?"  Part="1"
+AR Path="/5F3218EE/5F35FEA1" Ref="U4"  Part="1"
+F 0 "U4" H 3250 5942 50  0000 C CNN
+F 1 "MCP1700-3302E_SOT23" H 3250 5851 50  0000 C CNN
+F 2 "Package_TO_SOT_SMD:SOT-23" H 3250 5925 50  0001 C CNN
+F 3 "http://ww1.microchip.com/downloads/en/DeviceDoc/20001826D.pdf" H 3250 5700 50  0001 C CNN
+	1    3250 5700
+	1    0    0    -1
+$EndComp
+$Comp
+L power:GND #PWR0109
+U 1 1 5F3688B9
+P 3250 6150
+F 0 "#PWR0109" H 3250 5900 50  0001 C CNN
+F 1 "GND" H 3255 5977 50  0000 C CNN
+F 2 "" H 3250 6150 50  0001 C CNN
+F 3 "" H 3250 6150 50  0001 C CNN
+	1    3250 6150
+	1    0    0    -1
+$EndComp
+$Comp
+L power:+5V #PWR0111
+U 1 1 5F368EAD
+P 2650 5550
+F 0 "#PWR0111" H 2650 5400 50  0001 C CNN
+F 1 "+5V" H 2665 5723 50  0000 C CNN
+F 2 "" H 2650 5550 50  0001 C CNN
+F 3 "" H 2650 5550 50  0001 C CNN
+	1    2650 5550
+	1    0    0    -1
+$EndComp
+Wire Wire Line
+	2650 5700 2650 5550
+Connection ~ 2650 5700
+$Comp
+L power:+3.3VA #PWR0132
+U 1 1 5F36C949
+P 3750 5550
+F 0 "#PWR0132" H 3750 5400 50  0001 C CNN
+F 1 "+3.3VA" H 3765 5723 50  0000 C CNN
+F 2 "" H 3750 5550 50  0001 C CNN
+F 3 "" H 3750 5550 50  0001 C CNN
+	1    3750 5550
+	1    0    0    -1
+$EndComp
+Wire Wire Line
+	3750 5700 3750 5550
+Connection ~ 3750 5700
+$Comp
+L power:+3.3VA #PWR0139
+U 1 1 5F376205
+P 2850 3000
+F 0 "#PWR0139" H 2850 2850 50  0001 C CNN
+F 1 "+3.3VA" H 2865 3173 50  0000 C CNN
+F 2 "" H 2850 3000 50  0001 C CNN
+F 3 "" H 2850 3000 50  0001 C CNN
+	1    2850 3000
+	1    0    0    -1
+$EndComp
+$Comp
+L power:+3.3VA #PWR0165
+U 1 1 5F37902C
+P 5850 3100
+F 0 "#PWR0165" H 5850 2950 50  0001 C CNN
+F 1 "+3.3VA" H 5865 3273 50  0000 C CNN
+F 2 "" H 5850 3100 50  0001 C CNN
+F 3 "" H 5850 3100 50  0001 C CNN
+	1    5850 3100
+	1    0    0    -1
+$EndComp
+$Comp
+L power:+3.3VA #PWR0172
+U 1 1 5F384986
+P 8250 3550
+F 0 "#PWR0172" H 8250 3400 50  0001 C CNN
+F 1 "+3.3VA" H 8265 3723 50  0000 C CNN
+F 2 "" H 8250 3550 50  0001 C CNN
+F 3 "" H 8250 3550 50  0001 C CNN
+	1    8250 3550
+	1    0    0    -1
+$EndComp
+$Comp
+L power:+3.3VA #PWR0173
+U 1 1 5F38A5F4
+P 8400 5000
+F 0 "#PWR0173" H 8400 4850 50  0001 C CNN
+F 1 "+3.3VA" H 8415 5173 50  0000 C CNN
+F 2 "" H 8400 5000 50  0001 C CNN
+F 3 "" H 8400 5000 50  0001 C CNN
+	1    8400 5000
+	1    0    0    -1
+$EndComp
 $EndSCHEMATC

Commit message: cystal layout
Parts:
- added C27: 1uF, Capacitor_SMD:C_0402_1005Metric, symbol Device:C
- added C31: 100nF, Capacitor_SMD:C_0402_1005Metric, symbol Device:C
Connections:
- net +3.3VA: now also C27.1, C31.1
- net GND: now also C27.2, C31.2
Changed lines of the file:
@@
 	1    0    0    -1
 $EndComp
+$Comp
+L Device:C C?
+U 1 1 5F38F9CC
+P 4150 5850
+AR Path="/5F38F9CC" Ref="C?"  Part="1"
+AR Path="/5F569749/5F38F9CC" Ref="C?"  Part="1"
+AR Path="/5F3218EE/5F38F9CC" Ref="C27"  Part="1"
+F 0 "C27" H 4265 5896 50  0000 L CNN
+F 1 "1uF" H 4265 5805 50  0000 L CNN
+F 2 "Capacitor_SMD:C_0402_1005Metric" H 4188 5700 50  0001 C CNN
+F 3 "~" H 4150 5850 50  0001 C CNN
+	1    4150 5850
+	1    0    0    -1
+$EndComp
+$Comp
+L Device:C C?
+U 1 1 5F39274C
+P 4550 5850
+AR Path="/5F39274C" Ref="C?"  Part="1"
+AR Path="/5F569749/5F39274C" Ref="C?"  Part="1"
+AR Path="/5F3218EE/5F39274C" Ref="C31"  Part="1"
+F 0 "C31" H 4665 5896 50  0000 L CNN
+F 1 "100nF" H 4665 5805 50  0000 L CNN
+F 2 "Capacitor_SMD:C_0402_1005Metric" H 4588 5700 50  0001 C CNN
+F 3 "~" H 4550 5850 50  0001 C CNN
+	1    4550 5850
+	1    0    0    -1
+$EndComp
+Wire Wire Line
+	3750 5700 4150 5700
+Connection ~ 4150 5700
+Wire Wire Line
+	4150 5700 4550 5700
+Wire Wire Line
+	4550 6000 4150 6000
+Connection ~ 3750 6000
+Connection ~ 4150 6000
+Wire Wire Line
+	4150 6000 3750 6000
 $EndSCHEMATC
