File: drone_v3/_autosave-drone_v3.kicad_pcb (KiCad board)
At the start: 2 copper layers, 47.5 x 47.5 mm, 87 parts, among them J1 USB_B_Micro, J10 Conn_01x08_Male, J12 Conn_01x08_Male, J13 Conn_01x08_Male, J14 Conn_01x02_Male, J15 UART4_con, J16 Conn_01x03_Male, J17 Conn_01x02_Male, J18 Conn_01x03_Male, J19 Micro_SD_Card, J2 Conn_01x10_Female, J3 UART4_con, J4 Conn_01x04_Male, J5 Conn_01x02_Female, J6 Conn_01x04_Male, J7 Conn_01x04_Male, J8 UART4_con, J9 Conn_01x06_Male, Q1 2N3904, Q2 2N3904, SW1 SW_Push, U1 STM32F405RGTx, U2 USBLC6-2SC6, U3 MPU-9250, U4 MCP1700-3302E_SOT23, U5 24LC512, U6 NRF24L01_Breakout, U7 MS5611-01BA, U8 ICM-20602, U9 MCP1700-3302E_SOT23, Y1 Crystal_GND24

Commit message: crystal layout
Parts:
- C10, C14: moved to B.Cu
- moved C10 1.23 mm to (121.5, 108.0)
- moved C14 0.23 mm to (122.2, 108.0)
Connections:
- J1 pad 6: GND -> Net-(J1-Pad6)
- U1 pad 10: Net-(U1-Pad10) -> ADC1
- U1 pad 9: ADC1 -> Net-(U1-Pad9)
Routing:
- net GND: track 479.4 -> 495.6 mm, vias 311 -> 313
- net Net-(J1-Pad6): track 0.00 -> 7.21 mm
- net Net-(C4-Pad1): track 0.64 -> 4.69 mm
- net LED3: track 6.55 -> 7.54 mm
- net SD_MISO: track 23.8 -> 24.5 mm
- net VCC: track 320.4 -> 320.7 mm, vias 19 -> 21
