File: drone_v3/_autosave-IMU.sch (KiCad schematic (older format))
At the start: 22 parts, among them J2 Conn_01x10_Female, U10 ICM-20948, U3 MPU-9250, U4 MCP1700-3302E_SOT23, U8 MCP1804x-1802xDB

Commit message: change 20602 to 20948, ms5611 to bmp180
Parts:
- gave numbers to parts that had none: 1
Changed lines of the file:
@@
 $EndComp
 $Comp
-L Sensor_Pressure:BMP280 U?
+L Sensor_Pressure:BMP280 U7
 U 1 1 5F412E16
 P 8300 5650
-F 0 "U?" H 8530 5746 50  0000 L CNN
+F 0 "U7" H 8530 5746 50  0000 L CNN
 F 1 "BMP280" H 8530 5655 50  0000 L CNN
 F 2 "Package_LGA:Bosch_LGA-8_2x2.5mm_P0.65mm_ClockwisePinNumbering" H 8300 4950 50  0001 C CNN
