File: drone_v3/drone_v3.kicad_pcb (KiCad board)
At the start: 2 copper layers, 47.5 x 47.5 mm, 94 parts, among them J1 USB_B_Micro, J14 Conn_01x02_Male, J19 Micro_SD_Card, J2 Conn_01x10_Female, J7 Conn_01x04_Male, J9 Conn_01x06_Male, Q1 2N3904, Q2 2N3904, U3 MPU-9250, U7 BMP388, U9 MCP1700-3302E_SOT23, Y1 Crystal_GND24

Commit message: add
Routing:
- net IMU_CS: track 3.82 -> 9.31 mm
- net GND: track 655.6 -> 659.8 mm, vias 328 -> 321
- net IMU_INT: track 18.7 -> 22.4 mm
- net IMU_CS3: track 16.2 -> 19.0 mm
- net IMU_MOSI: track 39.0 -> 40.7 mm
- net IMU_MISO: track 43.9 -> 44.5 mm

Commit message: fix alot
Parts:
- C6: value VCAP -> CP
- J4: renamed from 3.3 RX1 TX1 GND
- J6: renamed from 3.3 CLK DIO GND
- moved C32 0.35 mm to (122.2, 91.7)
- moved C5 0.28 mm to (132.0, 114.7)
- moved R11 0.25 mm to (123.8, 94.7)
- moved R10 0.23 mm to (122.2, 94.7)
- renumbered PWR to D5, PWM to J10, GND to J12, 5v to J13, I2C to J15, SBUS to J16, Buzzer to J17, BOOT to J18, UART4 to J3, BAT to J5, UART3 to J8, 1k to R10, NRST to SW1, STM32F405 to U1, ICM-20948 to U10, ESD to U2, MCP1700 to U4, 24LC512 to U5, nRF24 to U6, MCP1804 to U8
Connections:
- C28 pad 1: +5V -> VBUS
- D6 pad 1: Net-(D6-Pad1) -> VBUS
- J1 pad 1: Net-(D6-Pad1) -> VBUS
- J2 pad 9: IMU1_CS -> IMU_CS3
- U2 pad 5: +5V -> VBUS
- U7 pad 6: IMU_CS3 -> IMU1_CS
Routing:
- net +5V: track 24.9 -> 41.3 mm
- net IMU1_CS: track 29.1 -> 17.9 mm, vias 1 -> 2
- net IMU_CS3: track 19.0 -> 30.0 mm, vias 2 -> 1
- net VBUS: track 0.00 -> 9.58 mm, vias 0 -> 2
- net IMU_MOSI: track 40.7 -> 45.2 mm
- net GND: track 659.8 -> 656.2 mm, vias 321 -> 312
- net Net-(D6-Pad1): track 3.26 -> 0.00 mm, vias 2 -> 0
- net IMU_INT: track 22.4 -> 23.7 mm
- net IMU_MISO: track 44.5 -> 43.2 mm
- net IMU_CLK: track 38.1 -> 38.9 mm
- net VCC: track 325.7 -> 324.8 mm
- net I2C_SCl: track 21.1 -> 21.9 mm
- net UART1_RX: track 12.1 -> 12.7 mm
Other:
- net class Default: clearance 0.2 -> 0.15
- rule trace_clearance: 0.2 -> 0.15
- rule via_min_size: 0.4 -> 0.5
