File: drone_v3/drone_v3.kicad_pcb (KiCad board)
At the start: 2 copper layers, 47.5 x 47.5 mm, 94 parts, among them J1 USB_B_Micro, J14 Conn_01x02_Male, J2 Conn_01x10_Female, J7 Conn_01x04_Male, Q1 2N3904, Q2 2N3904, U3 MPU-9250, U7 BMP388, Y1 Crystal_GND24

Commit message: update genber
Routing:
- net GND: track 722.1 -> 693.8 mm, vias 304 -> 303
- net IMU_CLK: track 38.9 -> 37.5 mm
- net IMU1_CS: track 17.9 -> 18.7 mm
- net IMU_CS2: track 16.9 -> 17.6 mm
- net IMU_MOSI: track 45.0 -> 45.7 mm
Other:
- net class USB: via_dia 0.5 -> 0.6
- rule via_min_size: 0.5 -> 0.6

Commit message: add alot
Parts:
- removed C12: 100n, Capacitor_SMD:C_0603_1608Metric_Pad1.05x0.95mm_HandSolder
- C6: value VCAP -> CP
- J4: renamed from 3.3v RX1 TX1 GND
- J6: renamed from 3.3v CLK DIO GND
- U10: renamed from ICM 20948
- moved G*** 2.60 mm to (123.0, 103.7)
- renumbered CAP to C5, PWR to D5, PWM to J10, GND to J12, 5v to J13, I2C1 to J15, SBUS to J16, BUZZ to J17, BOOT to J18, MicroSD to J19, UART4 to J3, BAT to J5, UART3 to J8, Telemetry to J9, 1k to R10, RST to SW1, STM32F405 to U1, ESD to U2, MCP1700 to U4, 24LC512 to U5, nRF24 to U6, MCP1804 to U8, MCP1700 to U9
Connections:
- J10 pad 8: USB_D+ -> Net-(J10-Pad8)
Routing:
- net GND: track 693.8 -> 717.0 mm, vias 303 -> 305
- net VCC: track 325.0 -> 322.1 mm, vias 20 -> 18
- net IMU_MOSI: track 45.7 -> 42.9 mm
- net IMU_INT: track 23.4 -> 24.1 mm
