File: drone_v3/MCU.sch (KiCad schematic (older format))
At the start: 15 parts, among them J18 Conn_01x03_Male, SW1 SW_Push, Y1 Crystal_GND24

Commit message: add alot
Connections:
- net GND: now also C9.2
- net VCC: now also C9.1
Other:
- moved on the sheet: C9
Changed lines of the file:
@@
 	5700 6300 7900 6300
 Wire Notes Line
-	7900 6300 7900 4850
+	8450 6350 8450 4900
 Wire Notes Line
 	7900 4850 5700 4850
@@
 L Device:C C?
 U 1 1 5F49F4ED
-P 6100 5550
+P 8000 5550
 AR Path="/5F49F4ED" Ref="C?"  Part="1"
 AR Path="/5F4758EB/5F49F4ED" Ref="C9"  Part="1"
-F 0 "C9" H 6215 5596 50  0000 L CNN
-F 1 "1u" H 6215 5505 50  0000 L CNN
-F 2 "Capacitor_SMD:C_0603_1608Metric_Pad1.05x0.95mm_HandSolder" H 6138 5400 50  0001 C CNN
-F 3 "~" H 6100 5550 50  0001 C CNN
-	1    6100 5550
+F 0 "C9" H 8115 5596 50  0000 L CNN
+F 1 "1u" H 8115 5505 50  0000 L CNN
+F 2 "Capacitor_SMD:C_0603_1608Metric_Pad1.05x0.95mm_HandSolder" H 8038 5400 50  0001 C CNN
+F 3 "~" H 8000 5550 50  0001 C CNN
+	1    8000 5550
 	1    0    0    -1
 $EndComp
@@
 Wire Wire Line
 	4600 5800 4600 5700
+Wire Wire Line
+	7650 5400 8000 5400
+Wire Wire Line
+	8000 5700 7650 5700
+Connection ~ 7650 5700
 $EndSCHEMATC

Commit message: cystal layout
Parts:
- C10, C12, C13, C14, C8, C9: footprint Capacitor_SMD:C_0603_1608Metric_Pad1.05x0.95mm_HandSolder -> Capacitor_SMD:C_0402_1005Metric
- C5, C6: footprint Capacitor_Tantalum_SMD:CP_EIA-2012-15_AVX-P_Pad1.30x1.05mm_HandSolder -> Capacitor_SMD:C_1206_3216Metric
Changed lines of the file:
@@
 F 0 "C10" H 6415 5596 50  0000 L CNN
 F 1 "100n" H 6415 5505 50  0000 L CNN
-F 2 "Capacitor_SMD:C_0603_1608Metric_Pad1.05x0.95mm_HandSolder" H 6338 5400 50  0001 C CNN
+F 2 "Capacitor_SMD:C_0402_1005Metric" H 6338 5400 50  0001 C CNN
 F 3 "~" H 6300 5550 50  0001 C CNN
 	1    6300 5550
@@
 F 0 "C12" H 6865 5596 50  0000 L CNN
 F 1 "100n" H 6865 5505 50  0000 L CNN
-F 2 "Capacitor_SMD:C_0603_1608Metric_Pad1.05x0.95mm_HandSolder" H 6788 5400 50  0001 C CNN
+F 2 "Capacitor_SMD:C_0402_1005Metric" H 6788 5400 50  0001 C CNN
 F 3 "~" H 6750 5550 50  0001 C CNN
 	1    6750 5550
@@
 F 0 "C13" H 7265 5596 50  0000 L CNN
 F 1 "100n" H 7265 5505 50  0000 L CNN
-F 2 "Capacitor_SMD:C_0603_1608Metric_Pad1.05x0.95mm_HandSolder" H 7188 5400 50  0001 C CNN
+F 2 "Capacitor_SMD:C_0402_1005Metric" H 7188 5400 50  0001 C CNN
 F 3 "~" H 7150 5550 50  0001 C CNN
 	1    7150 5550
@@
 F 0 "C14" H 7765 5596 50  0000 L CNN
 F 1 "1u" H 7765 5505 50  0000 L CNN
-F 2 "Capacitor_SMD:C_0603_1608Metric_Pad1.05x0.95mm_HandSolder" H 7688 5400 50  0001 C CNN
+F 2 "Capacitor_SMD:C_0402_1005Metric" H 7688 5400 50  0001 C CNN
 F 3 "~" H 7650 5550 50  0001 C CNN
 	1    7650 5550
@@
 F 0 "C8" H 5915 5596 50  0000 L CNN
 F 1 "100n" H 5915 5505 50  0000 L CNN
-F 2 "Capacitor_SMD:C_0603_1608Metric_Pad1.05x0.95mm_HandSolder" H 5838 5400 50  0001 C CNN
+F 2 "Capacitor_SMD:C_0402_1005Metric" H 5838 5400 50  0001 C CNN
 F 3 "~" H 5800 5550 50  0001 C CNN
 	1    5800 5550
@@
 F 0 "C9" H 8115 5596 50  0000 L CNN
 F 1 "1u" H 8115 5505 50  0000 L CNN
-F 2 "Capacitor_SMD:C_0603_1608Metric_Pad1.05x0.95mm_HandSolder" H 8038 5400 50  0001 C CNN
+F 2 "Capacitor_SMD:C_0402_1005Metric" H 8038 5400 50  0001 C CNN
 F 3 "~" H 8000 5550 50  0001 C CNN
 	1    8000 5550
@@
 F 0 "C5" V 5055 5500 50  0000 C CNN
 F 1 "CP" V 4964 5500 50  0000 C CNN
-F 2 "Capacitor_Tantalum_SMD:CP_EIA-2012-15_AVX-P_Pad1.30x1.05mm_HandSolder" H 4838 5350 50  0001 C CNN
+F 2 "Capacitor_SMD:C_1206_3216Metric" H 4838 5350 50  0001 C CNN
 F 3 "~" H 4800 5500 50  0001 C CNN
 	1    4800 5500
@@
 F 0 "C6" H 4918 5846 50  0000 L CNN
 F 1 "CP" H 4918 5755 50  0000 L CNN
-F 2 "Capacitor_Tantalum_SMD:CP_EIA-2012-15_AVX-P_Pad1.30x1.05mm_HandSolder" H 4838 5650 50  0001 C CNN
+F 2 "Capacitor_SMD:C_1206_3216Metric" H 4838 5650 50  0001 C CNN
 F 3 "~" H 4800 5800 50  0001 C CNN
 	1    4800 5800

Commit message: add alot
Parts:
- removed C12: 100n, Capacitor_SMD:C_0402_1005Metric, symbol Device:C
Changed lines of the file:
@@
-$Comp
-L Device:C C?
-U 1 1 5F49F4B2
-P 6750 5550
-AR Path="/5F49F4B2" Ref="C?"  Part="1"
-AR Path="/5F4758EB/5F49F4B2" Ref="C12"  Part="1"
-F 0 "C12" H 6865 5596 50  0000 L CNN
-F 1 "100n" H 6865 5505 50  0000 L CNN
-F 2 "Capacitor_SMD:C_0402_1005Metric" H 6788 5400 50  0001 C CNN
-F 3 "~" H 6750 5550 50  0001 C CNN
-	1    6750 5550
-	1    0    0    -1
-$EndComp
 $Comp
 L Device:C C?
@@
 Connection ~ 7650 5400
 Connection ~ 6300 5400
-Wire Wire Line
-	6300 5400 6750 5400
-Connection ~ 6750 5400
-Wire Wire Line
-	6750 5400 7150 5400
 Connection ~ 7150 5400
 Wire Wire Line
@@
 	8000 5700 7650 5700
 Connection ~ 7650 5700
+Wire Wire Line
+	6300 5400 7150 5400
 $EndSCHEMATC
